File: design_files/AST1021.brd (EAGLE design)
At the start: 10 x 10 mm, 10 parts, among them J1 SM05B, U1 PCT2075

Commit message: name change
Parts:
- C2: value 10uF -> 1uF
- J1: device tinycircuits:JST_SH_5X1 -> tinycircuits:JST_SH_5X1_EDGE
- R1: value 10.0K -> 1.00K
- R2: value 0.0 -> 1.00K
- R4: value 1.00K -> 10.0K
- moved R4 7.12 mm to (24.4, 13.2)
- moved R5 6.80 mm to (23.8, 14.8), turned to 180 degrees
- moved R1 6.22 mm to (21.7, 18.8)
- moved R2 5.52 mm to (20.0, 18.8), turned to 270 degrees
- moved R3 3.40 mm to (18.3, 18.8)
- moved C2 0.10 mm to (15.8, 13.4)
Connections:
- net GND: now also R1.1, R2.1; no longer R4.1, R5.1
- net GPIO1: now also R4.1, R5.1; no longer R1.1, R2.1
- net INT: now also R5.2; no longer R2.2
- net N$1: now also R1.2; no longer R3.2
- net N$2: now also R2.2; no longer R4.2
- net N$5: now also R3.2; no longer R5.2
- net VCC: now also R4.2; no longer R1.2
Other:
- board text added: "Wireling Temp Sensor"
- board text removed: "Temperature Sensor Board"
Changed lines of the file:
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@@
 <layer number="59" name="Invisible" color="7" fill="1" visible="no" active="no"/>
 <layer number="61" name="stand" color="7" fill="1" visible="no" active="no"/>
+<layer number="88" name="SimResults" color="9" fill="1" visible="yes" active="yes"/>
+<layer number="89" name="SimProbes" color="9" fill="1" visible="yes" active="yes"/>
 <layer number="90" name="Modules" color="5" fill="1" visible="yes" active="yes"/>
 <layer number="91" name="Nets" color="2" fill="1" visible="no" active="no"/>
@@
 <layer number="158" name="bResistor" color="7" fill="1" visible="no" active="yes"/>
 <layer number="159" name="henwayCAP" color="13" fill="1" visible="yes" active="yes"/>
+<layer number="160" name="IDFDebug" color="7" fill="1" visible="yes" active="yes"/>
 <layer number="191" name="mNets" color="7" fill="1" visible="no" active="no"/>
 <layer number="192" name="mBusses" color="7" fill="1" visible="no" active="no"/>
@@
 <wire x1="0" y1="40.8" x2="0" y2="0" width="0.127" layer="48"/>
 <dimension x1="15" y1="20" x2="25" y2="20" x3="20" y3="21.454653125" layer="48"/>
-<text x="38.111025" y="4.365003125" size="0.889" layer="48">Temperature Sensor Board</text>
+<text x="38.111025" y="4.365003125" size="0.889" layer="48">Wireling Temp Sensor</text>
 <text x="34.986825" y="1.7714" size="0.889" layer="48">AS-PCB-AST1021</text>
 <text x="57.3810375" y="1.6952" size="0.889" layer="48">2</text>
@@
 <attribute name="VALUE" value="0.1uF" x="16.4" y="15.9" size="1.778" layer="27" rot="R180" display="off"/>
 </element>
-<element name="C2" library="tinycircuits" package="C0603" value="10uF" x="15.7" y="13.4" rot="R90">
-<attribute name="PARTNO" value="AS-ITM-00002" x="15.7" y="13.4" size="1.778" layer="27" rot="R90" display="off"/>
-<attribute name="VALUE" value="10uF" x="15.7" y="13.4" size="1.778" layer="27" rot="R90" display="off"/>
+<element name="C2" library="tinycircuits" package="C0603" value="1uF" x="15.8" y="13.4" rot="R90">
+<attribute name="PARTNO" value="AS-ITM-00410" x="15.8" y="13.4" size="1.778" layer="27" rot="R90" display="off"/>
+<attribute name="VALUE" value="1uF" x="15.8" y="13.4" size="1.778" layer="27" rot="R90" display="off"/>
 </element>
-<element name="J1" library="tinycircuits" package="JST_SH_5X1" value="SM05B" x="20" y="12.125">
+<element name="J1" library="tinycircuits" package="JST_SH_5X1_EDGE" value="SM05B" x="20" y="12.125">
 <attribute name="PARTNO" value="AS-ITM-00340" x="20" y="12.125" size="1.778" layer="27" display="off"/>
 <attribute name="VALUE" value="SM05B" x="20" y="12.125" size="1.778" layer="27" display="off"/>
 <attribute name="PNPROTATION" value="180" x="20" y="12.125" size="1.778" layer="27" display="off"/>
 </element>
-<element name="R2" library="tinycircuits" package="0402" value="0.0" x="23.8" y="14.8" rot="R180">
-<attribute name="PARTNO" value="AS-ITM-00076" x="23.8" y="14.8" size="1.778" layer="27" rot="R180" display="off"/>
-<attribute name="VALUE" value="0.0" x="23.8" y="14.8" size="1.778" layer="27" rot="R180" display="off"/>
+<element name="R5" library="tinycircuits" package="0402" value="1.00K" x="23.8" y="14.8" rot="R180">
+<attribute name="PARTNO" value="AS-ITM-00003" x="23.8" y="14.8" size="1.778" layer="27" rot="R180" display="off"/>
+<attribute name="VALUE" value="1.00K" x="23.8" y="14.8" size="1.778" layer="27" rot="R180" display="off"/>
 </element>
-<element name="R1" library="tinycircuits" package="0402" value="10.0K" x="24.4" y="13.2" rot="R270">
+<element name="R4" library="tinycircuits" package="0402" value="10.0K" x="24.4" y="13.2" rot="R270">
 <attribute name="PARTNO" value="AS-ITM-00032" x="24.4" y="13.2" size="1.778" layer="27" rot="R270" display="off"/>
 <attribute name="VALUE" value="10.0K" x="24.4" y="13.2" size="1.778" layer="27" rot="R270" display="off"/>
@@
 <attribute name="VALUE" value="PCT2075" x="20" y="16.6" size="1.778" layer="27" rot="R90" display="off"/>
 </element>
-<element name="R3" library="tinycircuits" package="0402" value="1.00K" x="21.7" y="18.8" rot="R270">
+<element name="R1" library="tinycircuits" package="0402" value="1.00K" x="21.7" y="18.8" rot="R270">
 <attribute name="PARTNO" value="AS-ITM-00003" x="21.7" y="18.8" size="1.778" layer="27" rot="R270" display="off"/>
 <attribute name="VALUE" value="1.00K" x="21.7" y="18.8" size="1.778" layer="27" rot="R270" display="off"/>
 </element>
-<element name="R4" library="tinycircuits" package="0402" value="1.00K" x="20" y="18.8" rot="R270">
+<element name="R2" library="tinycircuits" package="0402" value="1.00K" x="20" y="18.8" rot="R270">
 <attribute name="PARTNO" value="AS-ITM-00003" x="20" y="18.8" size="1.778" layer="27" rot="R270" display="off"/>
 <attribute name="VALUE" value="1.00K" x="20" y="18.8" size="1.778" layer="27" rot="R270" display="off"/>
 </element>
-<element name="R5" library="tinycircuits" package="0402" value="1.00K" x="18.3" y="18.8" rot="R270">
+<element name="R3" library="tinycircuits" package="0402" value="1.00K" x="18.3" y="18.8" rot="R270">
 <attribute name="PARTNO" value="AS-ITM-00003" x="18.3" y="18.8" size="1.778" layer="27" rot="R270" display="off"/>
 <attribute name="VALUE" value="1.00K" x="18.3" y="18.8" size="1.778" layer="27" rot="R270" display="off"/>
@@
 <contactref element="U1" pad="GND"/>
 <contactref element="U1" pad="4"/>
-<via x="24.5" y="17.6" extent="1-16" drill="0.381"/>
+<via x="24.4" y="17.4" extent="1-16" drill="0.381"/>
 <via x="17" y="14" extent="1-16" drill="0.381"/>
 <via x="22.9" y="13.4" extent="1-16" drill="0.381"/>
+<contactref element="R1" pad="1"/>
+<contactref element="R2" pad="1"/>
 <contactref element="R3" pad="1"/>
-<contactref element="R4" pad="1"/>
-<contactref element="R5" pad="1"/>
 <wire x1="21.7" y1="19.4" x2="20" y2="19.4" width="0.2032" layer="1"/>
 <wire x1="20" y1="19.4" x2="18.3" y2="19.4" width="0.2032" layer="1"/>
@@
 <signal name="VCC">
 <contactref element="J1" pad="2"/>
-<contactref element="R1" pad="2"/>
+<contactref element="R4" pad="2"/>
 <contactref element="C2" pad="1"/>
 <contactref element="C1" pad="1"/>
@@
 <wire x1="19" y1="12.6" x2="24.4" y2="12.6" width="0.254" layer="1"/>
 <wire x1="19" y1="12.6" x2="15.75" y2="12.6" width="0.254" layer="1"/>
-<wire x1="15.75" y1="12.6" x2="15.7" y2="12.55" width="0.254" layer="1"/>
+<wire x1="15.75" y1="12.6" x2="15.8" y2="12.55" width="0.254" layer="1"/>
 <wire x1="18.9" y1="14.7" x2="19" y2="14.6" width="0.254" layer="1"/>
 <wire x1="18.6" y1="15.85" x2="16.9" y2="15.85" width="0.254" layer="1"/>
@@
 </signal>
 <signal name="INT">
-<contactref element="R2" pad="2"/>
+<contactref element="R5" pad="2"/>
 <contactref element="J1" pad="5"/>
 <wire x1="23.2" y1="14.8" x2="22.2" y2="14.8" width="0.254" layer="1"/>
@@
 </signal>
 <signal name="GPIO1">
-<contactref element="R2" pad="1"/>
-<contactref element="R1" pad="1"/>
+<contactref element="R5" pad="1"/>
+<contactref element="R4" pad="1"/>
 <contactref element="U1" pad="3"/>
 <wire x1="21.4" y1="16.85" x2="23.85" y2="16.85" width="0.254" layer="1"/>
@@
 <signal name="N$2">
 <contactref element="U1" pad="6"/>
-<contactref element="R4" pad="2"/>
+<contactref element="R2" pad="2"/>
 <wire x1="20" y1="18.2" x2="19.3" y2="18.2" width="0.2032" layer="1"/>
 <wire x1="19.3" y1="18.2" x2="19.2" y2="18.3" width="0.2032" layer="1"/>
@@
 <signal name="N$5">
 <contactref element="U1" pad="5"/>
-<contactref element="R5" pad="2"/>
+<contactref element="R3" pad="2"/>
 <wire x1="18.6" y1="17.35" x2="18.6" y2="18" width="0.2032" layer="1"/>
 <wire x1="18.6" y1="18" x2="18.3" y2="18.2" width="0.2032" layer="1"/>
@@
 <signal name="N$1">
 <contactref element="U1" pad="7"/>
-<contactref element="R3" pad="2"/>
+<contactref element="R1" pad="2"/>
 <wire x1="21.7" y1="18.2" x2="21" y2="18.2" width="0.2032" layer="1"/>
 <wire x1="21" y1="18.2" x2="20.9" y2="18.3" width="0.2032" layer="1"/>
