File: design_files/AST1021.sch (EAGLE design)
At the start: 9 parts, among them J1 SM05B, U1 PCT2075

Commit message: name change
Parts:
- C2: value 10uF -> 1uF; device tinycircuits:AS-ITM-00002 -> tinycircuits:AS-ITM-00410; PARTNO (none) -> AS-ITM-00410; VALUE (none) -> 1uF
- J1: device tinycircuits:AS-ITM-00340 -> tinycircuits:AS-ITM-00340EDGE
- R1: value 10.0K -> 1.00K; device tinycircuits:AS-ITM-00032 -> tinycircuits:AS-ITM-00003; PARTNO (none) -> AS-ITM-00003; VALUE (none) -> 1.00K
- R2: value 0.0 -> 1.00K; device tinycircuits:AS-ITM-00076 -> tinycircuits:AS-ITM-00003; PARTNO (none) -> AS-ITM-00003; VALUE (none) -> 1.00K
- R4: value 1.00K -> 10.0K; device tinycircuits:AS-ITM-00003 -> tinycircuits:AS-ITM-00032; PARTNO AS-ITM-00003 -> (none); VALUE 1.00K -> (none)
Connections:
- net GND: now also R1.1, R2.1; no longer R4.1, R5.1
- net GPIO1: now also R4.1, R5.1; no longer R1.1, R2.1
- net INT: now also R5.2; no longer R2.2
- net N$1: now also R1.2; no longer R3.2
- net N$2: now also R2.2; no longer R4.2
- net N$5: now also R3.2; no longer R5.2
- net VCC: now also R4.2; no longer R1.2
Other:
- note added: "Variant: Standard - R"
- note added: "Wireling Temp Sensor"
- note removed: "***Cut traces on bottom to Change Address"
- note removed: "Proto"
- note removed: "Temperature Sensor Board"
- note removed: "Variant: Standard"
- moved on the sheet: R1, R2, R3, R4, R5
